File: hw/R2P_DCM_module.sch (EAGLE design)
At the start: 53 parts, among them Q1 MOSFET-NCHANNELFDD8580, Q2 MOSFET-NCHANNELFDD8580, Q3 MOSFET-NCHANNELFDD8580, Q4 MOSFET-NCHANNELFDD8580, U1 STM32F103CX, U5 LD3985XX, X1 MICROMATCH-4, X2 OSC-XTAL212M_

Commit message: Removed misplaced via and disconnected MAX3051 shutdown pin
Connections:
- net +3V3: no longer SOT1.SHDN
Changed lines of the file:
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@@
 <part name="GND5" library="supply1" deviceset="GND" device=""/>
 <part name="GND6" library="supply1" deviceset="GND" device=""/>
-<part name="+3V5" library="supply1" deviceset="+3V3" device=""/>
 <part name="GND15" library="supply1" deviceset="GND" device=""/>
 <part name="P+2" library="supply" deviceset="+5V" device=""/>
@@
 <instance part="GND5" gate="1" x="124.46" y="76.2"/>
 <instance part="GND6" gate="1" x="88.9" y="68.58"/>
-<instance part="+3V5" gate="G$1" x="88.9" y="96.52"/>
 <instance part="GND15" gate="1" x="88.9" y="114.3"/>
 <instance part="P+2" gate="1" x="88.9" y="129.54"/>
@@
 </segment>
 <segment>
-<wire x1="91.44" y1="83.82" x2="88.9" y2="83.82" width="0.1524" layer="91"/>
-<wire x1="88.9" y1="83.82" x2="88.9" y2="93.98" width="0.1524" layer="91"/>
-<pinref part="SOT1" gate="G$1" pin="SHDN"/>
-<pinref part="+3V5" gate="G$1" pin="+3V3"/>
-</segment>
-<segment>

Commit message: increased bootstrap capacitor value
Parts:
- C1, C3: value 100n -> 220n
Changed lines of the file:
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@@
 <?xml version="1.0" encoding="utf-8"?>
 <!DOCTYPE eagle SYSTEM "eagle.dtd">
-<eagle version="6.2">
+<eagle version="6.4">
 <drawing>
 <settings>
@@
 <part name="GND7" library="supply1" deviceset="GND" device=""/>
 <part name="GND8" library="supply1" deviceset="GND" device=""/>
-<part name="C1" library="rcl" deviceset="C-EU" device="C0603" value="100n"/>
-<part name="C3" library="rcl" deviceset="C-EU" device="C0603" value="100n"/>
+<part name="C1" library="rcl" deviceset="C-EU" device="C0603" value="220n"/>
+<part name="C3" library="rcl" deviceset="C-EU" device="C0603" value="220n"/>
 <part name="U$2" library="SparkFun" deviceset="ACS712" device=""/>
 <part name="GND23" library="supply1" deviceset="GND" device=""/>

Commit message: Corrected RDEAD value
Parts:
- R8: value 10 -> 10k
Changed lines of the file:
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@@
 <part name="GND9" library="supply1" deviceset="GND" device=""/>
 <part name="GND10" library="supply1" deviceset="GND" device=""/>
-<part name="R8" library="rcl" deviceset="R-EU_" device="R0603" value="10"/>
+<part name="R8" library="rcl" deviceset="R-EU_" device="R0603" value="10k"/>
 <part name="GND13" library="supply1" deviceset="GND" device=""/>
 <part name="+3V6" library="supply1" deviceset="+3V3" device=""/>
